File: KiKad/Jamma SuperGun CPS1 Harness/Jamma SuperGun CPS1 Harness.kicad_sch (KiCad schematic)
At the start: 2 parts

Commit message: updates
Parts:
- renumbered J_FEMALE to J_FEMALE1, J_MALE to J_MALE1
Connections:
- net +12V: now also J_FEMALE1.6, J_MALE1.6; no longer J_FEMALE1.06, J_MALE1.06
- net +5V: now also J_FEMALE1.3, J_FEMALE1.4, J_MALE1.3, J_MALE1.4; no longer J_FEMALE1.03, J_FEMALE1.04, J_MALE1.03, J_MALE1.04
- net -5V: now also J_FEMALE1.5, J_MALE1.5; no longer J_FEMALE1.05, J_MALE1.05
- net Coin Counter 1: now also J_FEMALE1.8, J_MALE1.8; no longer J_FEMALE1.08, J_MALE1.08
- net GND: now also J_FEMALE1.1, J_FEMALE1.2, J_MALE1.1, J_MALE1.2; no longer J_FEMALE1.01, J_FEMALE1.02, J_MALE1.01, J_MALE1.02
- net Lockout 1: now also J_FEMALE1.9, J_MALE1.9; no longer J_FEMALE1.09, J_MALE1.09
Changed lines of the file:
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@@
 		(dnp no)
 		(fields_autoplaced yes)
-		(property "Reference" "J_FEMALE"
+		(property "Reference" "J_FEMALE1"
 			(at 114.3 97.7899 0)
 			(show_name no)
@@
 		(pin "27"
 		)
-		(pin "09"
-		)
-		(pin "08"
-		)
-		(pin "06"
-		)
-		(pin "05"
-		)
-		(pin "04"
-		)
-		(pin "03"
-		)
-		(pin "02"
-		)
-		(pin "01"
+		(pin "3"
+		)
+		(pin "1"
+		)
+		(pin "5"
+		)
+		(pin "2"
+		)
+		(pin "4"
+		)
+		(pin "9"
+		)
+		(pin "8"
+		)
+		(pin "6"
 		)
 		(pin "10"
@@
 			(project "Jamma SuperGun CPS1 Harness"
 				(path "/f2e2e4d6-2af3-4060-b5a1-3dfdca0e7db5"
-					(reference "J_FEMALE")
+					(reference "J_FEMALE1")
 					(unit 1)
 				)
@@
 	)
 	(symbol
+		(lib_name "JAMMA_56_1")
 		(lib_id "kicad-symbol-library:JAMMA_56")
 		(at 31.75 20.32 0)
@@
 		(dnp no)
 		(fields_autoplaced yes)
-		(property "Reference" "J_MALE"
+		(property "Reference" "J_MALE1"
 			(at 69.85 97.7899 0)
 			(show_name no)
@@
 		(pin "27"
 		)
-		(pin "09"
-		)
-		(pin "08"
-		)
-		(pin "06"
-		)
-		(pin "05"
-		)
-		(pin "04"
-		)
-		(pin "03"
-		)
-		(pin "02"
-		)
-		(pin "01"
+		(pin "6"
+		)
+		(pin "3"
+		)
+		(pin "5"
+		)
+		(pin "1"
+		)
+		(pin "8"
+		)
+		(pin "9"
+		)
+		(pin "2"
+		)
+		(pin "4"
 		)
 		(pin "10"
@@
 			(project "Jamma SuperGun CPS1 Harness"
 				(path "/f2e2e4d6-2af3-4060-b5a1-3dfdca0e7db5"
-					(reference "J_MALE")
+					(reference "J_MALE1")
 					(unit 1)
 				)

Commit message: updates
Parts:
- added CPS1_KH1: (no value), symbol kicad-symbol-library:CPS1_KICK_HARNESS
Connections:
- net GND: now also CPS1_KH1.1, CPS1_KH1.2; no longer J_MALE1.27, J_MALE1.e
- net N/C: no longer J_MALE1.25, J_MALE1.26, J_MALE1.c, J_MALE1.d
- net 1P Button 1 renamed 1P_LP
- net 1P Button 2 renamed 1P_MP
- net 1P Button 3 renamed 1P_HP
- net 1P_HP: now also J_MALE1.26; no longer J_MALE1.24
- net 2P Button 1 renamed 2P_LP
- net 2P Button 2 renamed 2P_MP
- net 2P Button 3 renamed 2P_HP
- net 2P_HP: now also J_MALE1.d; no longer J_MALE1.b
- new net 1P_HK: CPS1_KH1.5, J_MALE1.27
- new net 1P_LK: CPS1_KH1.3, J_MALE1.24
- new net 1P_MK: CPS1_KH1.4, J_MALE1.25
- new net 2P_HK: CPS1_KH1.9, J_MALE1.e
- new net 2P_LK: CPS1_KH1.7, J_MALE1.b
- new net 2P_MK: CPS1_KH1.8, J_MALE1.c
Other:
- moved on the sheet: J_FEMALE1

Commit message: updates
Parts:
- CPS1_KH1: footprint (none) -> Connector_JST:JST_EH_B10B-EH-A_1x10_P2.50mm_Vertical
Changed lines of the file:
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@@
 			)
 		)
-		(property "Footprint" ""
+		(property "Footprint" "Connector_JST:JST_EH_B10B-EH-A_1x10_P2.50mm_Vertical"
 			(at 156.21 25.4 0)
 			(hide yes)
@@
 		(pin "9"
 		)
+		(pin "10"
+		)
+		(pin "6"
+		)
 		(instances

Commit message: fix warnings
Connections:
- removed net N/C: J_FEMALE1.25, J_FEMALE1.26, J_FEMALE1.c, J_FEMALE1.d
- no-connect marks 0 -> 6
Changed lines of the file:
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@@
 	(generator_version "10.0")
 	(paper "A4")
+	(no_connect
+		(at 127 165.1)
+	)
+	(no_connect
+		(at 127 162.56)
+	)
+	(no_connect
+		(at 162.56 40.64)
+	)
+	(no_connect
+		(at 162.56 50.8)
+	)
+	(no_connect
+		(at 127 88.9)
+	)
+	(no_connect
+		(at 127 91.44)
+	)
 	(wire
 		(pts
@@
 	(wire
 		(pts
-			(xy 104.14 88.9) (xy 127 88.9)
-		)
-		(stroke
-			(width 0)
-			(type default)
-		)
-	)
-	(wire
-		(pts
 			(xy 142.24 38.1) (xy 162.56 38.1)
 		)
@@
 	(wire
 		(pts
-			(xy 104.14 91.44) (xy 127 91.44)
-		)
-		(stroke
-			(width 0)
-			(type default)
-		)
-	)
-	(wire
-		(pts
 			(xy 38.1 104.14) (xy 60.96 104.14)
 		)
@@
 	(wire
 		(pts
-			(xy 104.14 162.56) (xy 127 162.56)
-		)
-		(stroke
-			(width 0)
-			(type default)
-		)
-	)
-	(wire
-		(pts
 			(xy 38.1 50.8) (xy 60.96 50.8)
 		)
@@
 		(pts
 			(xy 104.14 144.78) (xy 127 144.78)
-		)
-		(stroke
-			(width 0)
-			(type default)
-		)
-	)
-	(wire
-		(pts
-			(xy 104.14 165.1) (xy 127 165.1)
 		)
 		(stroke
@@
 		)
 	)
-	(label "N{slash}C"
-		(at 104.14 165.1 0)
-		(effects
-			(font
-				(size 1.27 1.27)
-			)
-			(justify left bottom)
-		)
-	)
 	(label "2P Up"
 		(at 104.14 144.78 0)
@@
 		)
 	)
-	(label "N{slash}C"
-		(at 104.14 162.56 0)
-		(effects
-			(font
-				(size 1.27 1.27)
-			)
-			(justify left bottom)
-		)
-	)
 	(label "Audio GND"
 		(at 104.14 127 0)
@@
 		)
 	)
-	(label "N{slash}C"
-		(at 104.14 91.44 0)
-		(effects
-			(font
-				(size 1.27 1.27)
-			)
-			(justify left bottom)
-		)
-	)
 	(label "Video Blue"
 		(at 104.14 58.42 0)
@@
 		(effects
 			(font
-				(size 1.27 1.27)
-			)
-			(justify left bottom)
-		)
-	)
-	(label "N{slash}C"
-		(at 104.14 88.9 0)
-		(effects
-			(font
