File: KiKad/Jamma SuperGun CPS1 Harness/Jamma SuperGun CPS1 Harness.kicad_pcb (KiCad board)
At the start: 2 copper layers, 111.5 x 36.9 mm, 3 parts

Commit message: fix warnings
Connections:
- J_FEMALE1 pad c: /N/C -> unconnected-(J_FEMALE1-Padc)
- J_FEMALE1 pad d: /N/C -> unconnected-(J_FEMALE1-Padd)
Routing:
- net /GND: track 202.2 -> 206.2 mm, vias 0 -> 2
- net /+5V: track 107.6 -> 111.6 mm, vias 0 -> 2
- net /-5V: vias 0 -> 1
- net /+12V: vias 0 -> 1
Changed lines of the file:
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@@
 			(size 2.35 8)
 			(layers "F.Mask" "B.Cu" "F.Paste")
-			(net "/N{slash}C")
+			(net "unconnected-(J_FEMALE1-Padc)")
 			(pinfunction "c_c")
-			(pintype "input")
+			(pintype "input+no_connect")
 		)
 		(pad "d" smd rect
@@
 			(size 2.35 8)
 			(layers "F.Mask" "B.Cu" "F.Paste")
-			(net "/N{slash}C")
+			(net "unconnected-(J_FEMALE1-Padd)")
 			(pinfunction "d_d")
-			(pintype "input")
+			(pintype "input+no_connect")
 		)
 		(pad "e" smd rect
@@
 			(net "unconnected-(CPS1_KH1-Pad6)")
 			(pinfunction "6_6")
-			(pintype "input")
+			(pintype "input+no_connect")
 		)
 		(pad "7" thru_hole oval
@@
 			(net "unconnected-(CPS1_KH1-Pad10)")
 			(pinfunction "10_10")
-			(pintype "input")
+			(pintype "input+no_connect")
 		)
 		(embedded_fonts no)
@@
 	)
 	(segment
+		(start 147.71 46)
+		(end 147.71 56.524)
+		(width 1)
+		(layer "F.Cu")
+		(net "/GND")
+	)
+	(segment
 		(start 143.8 48.5)
 		(end 143.75 48.55)
@@
 	)
 	(segment
+		(start 147.71 56.524)
+		(end 147.71 72.9)
+		(width 1)
+		(layer "F.Cu")
+		(net "/GND")
+	)
+	(segment
 		(start 245.922 60.08)
 		(end 243.422 60.08)
@@
 	)
 	(segment
-		(start 147.71 46)
-		(end 147.71 72.9)
+		(start 143.75 56.524)
+		(end 147.71 56.524)
 		(width 1)
 		(layer "F.Cu")
@@
 		(width 1)
 		(layer "F.Cu")
+		(net "/GND")
+	)
+	(via
+		(at 147.71 56.524)
+		(size 0.6)
+		(drill 0.3)
+		(layers "F.Cu" "B.Cu")
+		(net "/GND")
+	)
+	(via
+		(at 143.75 56.524)
+		(size 0.6)
+		(drill 0.3)
+		(layers "F.Cu" "B.Cu")
 		(net "/GND")
 	)
@@
 	)
 	(segment
+		(start 151.67 46)
+		(end 151.67 56.524)
+		(width 1)
+		(layer "F.Cu")
+		(net "/+5V")
+	)
+	(segment
+		(start 155.63 46)
+		(end 155.63 56.524)
+		(width 1)
+		(layer "F.Cu")
+		(net "/+5V")
+	)
+	(segment
+		(start 151.67 56.524)
+		(end 151.67 72.9)
+		(width 1)
+		(layer "F.Cu")
+		(net "/+5V")
+	)
+	(segment
+		(start 155.63 56.524)
+		(end 155.63 72.9)
+		(width 1)
+		(layer "F.Cu")
+		(net "/+5V")
+	)
+	(segment
+		(start 151.67 56.524)
+		(end 155.63 56.524)
+		(width 1)
+		(layer "F.Cu")
+		(net "/+5V")
+	)
+	(via
+		(at 151.67 56.524)
+		(size 0.6)
+		(drill 0.3)
+		(layers "F.Cu" "B.Cu")
+		(net "/+5V")
+	)
+	(via
+		(at 155.63 56.524)
+		(size 0.6)
+		(drill 0.3)
+		(layers "F.Cu" "B.Cu")
+		(net "/+5V")
+	)
+	(segment
 		(start 155.63 46)
 		(end 155.63 72.9)
 		(width 1)
-		(layer "F.Cu")
+		(layer "B.Cu")
 		(net "/+5V")
 	)
@@
 		(end 151.67 72.9)
 		(width 1)
-		(layer "F.Cu")
+		(layer "B.Cu")
 		(net "/+5V")
 	)
 	(segment
-		(start 155.63 46)
-		(end 155.63 72.9)
-		(width 1)
-		(layer "B.Cu")
-		(net "/+5V")
-	)
-	(segment
-		(start 151.67 46)
-		(end 151.67 72.9)
-		(width 1)
-		(layer "B.Cu")
-		(net "/+5V")
+		(start 159.6 56.524)
+		(end 159.6 72.375)
+		(width 1)
+		(layer "F.Cu")
+		(net "/-5V")
 	)
 	(segment
 		(start 159.6 48.025)
-		(end 159.6 72.375)
-		(width 1)
-		(layer "F.Cu")
+		(end 159.6 56.524)
+		(width 1)
+		(layer "F.Cu")
+		(net "/-5V")
+	)
+	(via
+		(at 159.6 56.524)
+		(size 0.6)
+		(drill 0.3)
+		(layers "F.Cu" "B.Cu")
 		(net "/-5V")
 	)
@@
 	)
 	(segment
+		(start 163.55 56.524)
+		(end 163.55 72.9)
+		(width 1)
+		(layer "F.Cu")
+		(net "/+12V")
+	)
+	(segment
 		(start 163.55 46)
-		(end 163.55 72.9)
+		(end 163.55 56.524)
 		(width 1)
 		(layer "F.Cu")
 		(net "/+12V")
 	)
+	(via
+		(at 163.55 56.524)
+		(size 0.6)
+		(drill 0.3)
+		(layers "F.Cu" "B.Cu")
+		(net "/+12V")
+	)

Commit message: minor changes
Parts:
- ARCADE BOARD: renamed from J_FEMALE1
- CPS1 KICK HARNESS: renamed from CPS1_KH1
- renumbered J_MALE1 to CABINET/SUPERGUN
Connections:
- ARCADE BOARD pad 25: /N/C -> unconnected-(J_FEMALE1-Pad25)
- ARCADE BOARD pad 26: /N/C -> unconnected-(J_FEMALE1-Pad26)
Changed lines of the file:
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@@
 		(layer "F.Cu")
 		(at 198.21 91.9)
-		(property "Reference" "J_FEMALE1"
-			(at -1 -13.3 0)
+		(property "Reference" "ARCADE BOARD"
+			(at -1 -25.216 0)
 			(layer "F.SilkS")
 			(effects
@@
 			(size 2.35 8)
 			(layers "F.Cu" "F.Mask" "F.Paste")
-			(net "/N{slash}C")
+			(net "unconnected-(J_FEMALE1-Pad25)")
 			(pinfunction "25_25")
-			(pintype "input")
+			(pintype "input+no_connect")
 		)
 		(pad "26" smd rect
@@
 			(size 2.35 8)
 			(layers "F.Cu" "F.Mask" "F.Paste")
-			(net "/N{slash}C")
+			(net "unconnected-(J_FEMALE1-Pad26)")
 			(pinfunction "26_26")
-			(pintype "input")
+			(pintype "input+no_connect")
 		)
 		(pad "27" smd rect
@@
 		(layer "F.Cu")
 		(at 198.21 65)
-		(property "Reference" "J_MALE1"
+		(property "Reference" "CABINET/SUPERGUN"
 			(at -1 -13.3 0)
 			(layer "F.SilkS")
@@
 		(descr "JST EH series connector, B10B-EH-A (http://www.jst-mfg.com/product/pdf/eng/eEH.pdf)")
 		(tags "connector JST EH vertical")
-		(property "Reference" "CPS1_KH1"
-			(at 11.25 -2.8 0)
+		(property "Reference" "CPS1 KICK HARNESS"
+			(at 11.25 3.302 0)
 			(layer "F.SilkS")
 			(effects

Commit message: labels
Other:
- board text added: "10 9 8 7 6 5 4 3 2 1"
- board text added: "Player 1"
- board text added: "Player 2"
- board text added: "_{HK} _{MK} _{LK}"
Changed lines of the file:
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@@
 		)
+	)
+	(gr_rect
+		(start 225.254 62.366)
+		(end 232.874 65.668)
+		(stroke
+			(width 0.1)
+			(type default)
+		)
+		(fill no)
+		(layer "F.SilkS")
+	)
+	(gr_rect
+		(start 235.414 62.366)
+		(end 243.034 65.668)
+		(stroke
+			(width 0.1)
+			(type default)
+		)
+		(fill no)
+		(layer "F.SilkS")
 	)
 	(gr_poly
@@
 		(layer "Edge.Cuts")
 	)
+	(gr_text "10  9  8  7  6  5  4  3  2  1"
+		(at 222.714 63.89 0)
+		(layer "F.SilkS")
+		(effects
+			(font
+				(size 1 1)
+				(thickness 0.15)
+			)
+			(justify left bottom)
+		)
+	)
+	(gr_text "_{HK} _{MK} _{LK}\n"
+		(at 225.762 65.16 0)
+		(layer "F.SilkS")
+		(effects
+			(font
+				(size 1 1)
+				(thickness 0.15)
+			)
+			(justify left bottom)
+		)
+	)
+	(gr_text "Player 2"
+		(at 225.762 67.192 0)
+		(layer "F.SilkS")
+		(effects
+			(font
+				(size 1 1)
+				(thickness 0.15)
+			)
+			(justify left bottom)
+		)
+	)
+	(gr_text "_{HK} _{MK} _{LK}"
+		(at 236.176 65.16 0)
+		(layer "F.SilkS")
+		(effects
+			(font
+				(size 1 1)
+				(thickness 0.15)
+			)
+			(justify left bottom)
+		)
+	)
+	(gr_text "Player 1"
+		(at 236.176 67.192 0)
+		(layer "F.SilkS")
+		(effects
+			(font
+				(size 1 1)
+				(thickness 0.15)
+			)
+			(justify left bottom)
+		)
+	)
 	(segment

Commit message: fix pads on the back
Other:
- board text added: "^{+12V}"
- board text added: "^{+5V}"
- board text added: "^{-5V}"
- board text added: "^{GND}"

Commit message: updates
Parts:
- CPS1 BOARD: renamed from ARCADE BOARD
Other:
- board text added: "KICK HARNESS ADAPTER"
- board text added: "^{B1}"
- board text added: "^{B2}"
- board text added: "^{B3}"
- board text added: "^{B4}"
- board text added: "^{B5}"
- board text added: "^{B6}"
- board text added: "^{HK}"
- board text added: "^{HP}"
- board text added: "^{LK}"
- board text added: "^{LP}"
- board text added: "^{MK}"
- board text added: "^{MP}"
- board text added: "_{B1} _{B2} _{B5}"
- board text added: "_{B3} _{B4} _{B6}"
- board text added: "_{LK} _{MK} _{HK}"
- board text added: "_{LP} _{MP} _{HP}"

Commit message: updates
Other:
- outline, holes or cut-outs redrawn
- board text added: "V1"
- board text added: "^{designed by talex-tnt}"
Changed lines of the file:
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@@
 	(gr_poly
 		(pts
-			(xy 141.434 78.368) (xy 252.94 78.368) (xy 252.94 42.554) (xy 252.178 41.5) (xy 142.45 41.5) (xy 141.434 42.554)
+			(xy 141.434 78.368) (xy 252.94 78.368) (xy 252.94 42.554) (xy 252.178 41.5) (xy 167.342 41.5) (xy 142.45 41.5)
+			(xy 141.434 42.554)
 		)
 		(stroke
@@
 		)
 	)
+	(gr_text "^{designed by talex-tnt}"
+		(at 178.264 63.89 0)
+		(layer "F.SilkS")
+		(effects
+			(font
+				(size 1.2 1.2)
+				(thickness 0.15)
+			)
+		)
+	)
 	(gr_text "KICK HARNESS ADAPTER"
 		(at 197.568 59.572 0)
 		(layer "F.SilkS")
 		(effects
+			(font
+				(size 1.2 1.2)
+				(thickness 0.15)
+			)
+		)
+	)
+	(gr_text "V1"
+		(at 197.568 61.858 0)
+		(layer "F.SilkS")
+		(effects
