File: KiKad/Jamma SuperGun CPS1 Harness/Jamma SuperGun CPS1 Harness.kicad_pcb (KiCad board)
At the start: 2 copper layers, 111.5 x 36.9 mm, 3 parts

Commit message: updates
Parts:
- ARCADE CABINET/SUPERGUN: renamed from CABINET/SUPERGUN
- CPS1 JAMMA EDGE: renamed from CPS1 BOARD
Other:
- outline, holes or cut-outs redrawn
